Commit message: updated for engg4480 lab2

File: teeterbot_description/urdf/teeterbot.urdf.xacro (robot description, xacro)
@@ -46,5 +46,5 @@
     </plugin>
   </gazebo>
-  <xacro:macro name="wheel" params="name y_offset" >
+  <xacro:macro name="wheel" params="name y_offset z_offset *link_pose">
     <link name="${name}" >
       <inertial>
@@ -54,5 +54,5 @@
       </inertial>
       <visual>
-        <origin xyz="0 0 0" rpy="0 0 0"/>
+        <origin xyz="0 0 ${z_offset}" rpy="0 0 0"/>
         <geometry>
           <cylinder radius="${wheel_radius}" length="${wheel_thickness}"/>
@@ -61,12 +61,12 @@
       </visual>
       <visual>
-        <origin xyz="0 0 0" rpy="1.5707 0 0"/>
+        <xacro:insert_block name="link_pose" />
         <geometry>
-          <cylinder radius="${wheel_thickness/2 + 0.01}" length="0.07"/>
+            <mesh filename="package://teeterbot_description/meshes/wheel.STL"/>
         </geometry>
         <material name="grey"/>
       </visual>
       <collision name="collision_${name}">
-        <origin xyz="0 0 0" rpy="0 0 0"/>
+        <origin xyz="0 0 ${z_offset}" rpy="0 0 0"/>
         <geometry>
           <cylinder radius="${wheel_radius}" length="${wheel_thickness}"/>
@@ -81,6 +81,10 @@
     </joint>
   </xacro:macro>
-  <wheel name="left_wheel" y_offset="${wheelbase/2}" />
-  <wheel name="right_wheel" y_offset="${-wheelbase/2}" />
+  <wheel name="left_wheel" y_offset="${wheelbase/2}" z_offset="-0.03" >
+    <origin xyz="0 0.06 -0.37" rpy="0 3.1415 0"/>
+  </wheel>
+  <wheel name="right_wheel" y_offset="${-wheelbase/2}" z_offset="0.03">
+    <origin xyz="0 0.06 0.37" rpy="0 0 0"/>
+  </wheel>
   <link name="body_com">
     <inertial>
@@ -90,8 +94,8 @@
     </inertial>
     <visual>
-      <origin xyz="0 0 0" rpy="0 0 0"/>
-      <geometry>
-        <box size="${body_depth} ${body_width} ${body_length}"/>
-      </geometry>
+      <origin xyz="0 0 -${body_length/2 - 0.051225}" rpy="0 0 0"/>
+        <geometry>
+            <mesh filename="package://teeterbot_description/meshes/base.STL"/>
+        </geometry>
       <material name="orange"/>
     </visual>
